File: ObsKeyBoardHw.kicad_sch (KiCad schematic)
At the start: 28 parts, among them SW01 RotaryEncoder_Switch, SW01 SW_Push, SW02 RotaryEncoder_Switch, SW02 SW_Push, SW03 SW_Push, SW04 SW_Push, SW10 RotaryEncoder_Switch, SW10 SW_Push, SW11 RotaryEncoder_Switch, SW11 SW_Push, SW12 RotaryEncoder_Switch, SW12 SW_Push, SW13 SW_Push, SW14 SW_Push, SW20 SW_Push, SW21 SW_Push, SW22 SW_Push, SW23 SW_Push, SW24 SW_Push, U1 ESP32-S2-WROVER

Commit message: 添加外壳
Parts:
- added C4: 22uF, Capacitor_SMD:C_0805_2012Metric, symbol Device:C_Small
- added C5: 0.1uF, Capacitor_SMD:C_0805_2012Metric, symbol Device:C_Small
- added C6, C7: 1uF, Capacitor_SMD:C_0805_2012Metric, symbol Device:C_Small
- added H1: (no value), symbol Mechanical:MountingHole
- added H2, H3, H4: MountingHole, MountingHole:MountingHole_3.2mm_M3_ISO7380, symbol Mechanical:MountingHole
- added R1, R2: 10K, Resistor_SMD:R_0805_2012Metric, symbol Device:R_Small
- added SW_BOOT1, SW_EN1: SW_Push, Button_Switch_SMD:SW_SPST_CK_RS282G05A3, symbol Switch:SW_Push
- C1: renamed from C?; value (none) -> 1uF; footprint (none) -> Capacitor_SMD:C_0805_2012Metric
- C3: renamed from C?; value (none) -> 22uF
- J1: renamed from J?; value (none) -> USB_B; footprint (none) -> Connector_USB:USB_B_Lumberg_2411_02_Horizontal
- RE0: renamed from SW00; value (none) -> RotaryEncoder_Switch; footprint (none) -> Rotary_Encoder:RotaryEncoder_Alps_EC11E-Switch_Vertical_H20mm
- SW0: renamed from SW00; value (none) -> SW_Push; footprint (none) -> Button_Switch_Keyboard:SW_Cherry_MX_1.00u_Plate
- U2: renamed from U?; value (none) -> AMS1117-3.3; footprint (none) -> Package_TO_SOT_SMD:SOT-223-3_TabPin2
- U3: renamed from U?; value (none) -> BC6561; footprint (none) -> Package_SO:SSOP-20_5.3x7.2mm_P0.65mm
- gave numbers to parts that had none: 1
- renumbered SW01 to RE1, SW10 to RE10, SW11 to RE11, SW12 to RE12, SW02 to RE2, SW01 to SW1, SW02 to SW2, SW03 to SW3, SW04 to SW4
Connections:
- net +3V3: now also U1.2 (3V3), U3.2 (VCC), C4.2, C5.2, C6.2, R1.1, R2.1
- net C0: now also U3.14 (C0)
- net C1: now also U3.15 (C1)
- net C2: now also U3.16 (C2)
- net C3: now also U3.17 (C3)
- net C4: now also U3.18 (C4)
- net EA_00: now also U1.6 (IO03)
- net EA_01: now also U1.8 (IO05)
- net EA_02: now also U1.10 (IO07)
- net EA_10: now also U1.16 (IO13)
- net EA_11: now also U1.18 (IO15)
- net EA_12: now also U1.20 (IO17)
- net EB_00: now also U1.7 (IO04)
- net EB_01: now also U1.9 (IO06)
- net EB_02: now also U1.11 (IO08)
- net EB_10: now also U1.17 (IO14)
- net EB_11: now also U1.19 (IO16)
- net EB_12: now also U1.21 (IO18)
- net GND: now also U1.1 (GND), U1.26 (GND), U1.42 (GND), U1.43 (GND), U3.13 (GND), C4.1, C5.1, C6.1, C7.1, SW_BOOT1.1, SW_EN1.1
- net R0: now also U3.3 (R0)
- net R1: now also U3.4 (R1)
- net R2: now also U3.5 (R2)
- net R3: now also U3.6 (R3)
- net R4: now also U3.7 (R4)
- net USB_D+: now also U1.23 (USB_D+)
- net USB_D-: now also U1.22 (USB_D-)
- net ESP_IO0: now reaches U1.3 (IO00)
- net ESP_IO0: now also R2.2, SW_BOOT1.2
- net K_TX: now reaches U1.4 (IO01)
- net K_TX: now also U3.12 (TX)
- net ESP_EN: now reaches U1.41 (EN)
- net ESP_EN: now also C7.2, R1.2, SW_EN1.2
- no-connect marks 0 -> 26
Other:
- moved on the sheet: U1, U3
